Commit message: Add files via upload

File: x80sv_description/urdf/x80sv.xacro (robot description, xacro)
@@ -1,4 +1,10 @@
 <?xml version='1.0' ?>
 <robot name="x80sv" xmlns:xacro="http://www.ros.org/wiki/xacro">
+	 <material name="Black">
+           <color rgba="0 0 0 1"/>
+         </material>
+	 <material name="gray">
+           <color rgba="0.8 0.8 0.8 1"/>
+         </material>
 	<xacro:include filename="$(find x80sv_description)/urdf/wheel.xacro" />
  <!--
@@ -14,5 +20,5 @@
 -->
 <xacro:property name="wheel_base" value="0.2" />
-<xacro:property name="wheel_diameter" value="0.16" />
+<xacro:property name="wheel_diameter" value="0.18" />
 <xacro:property name="wheel_distance" value="0.305"/>
 <xacro:property name="axis_height" value="0.05" />
@@ -36,5 +42,5 @@
 				<box size="0.001 0.001 0.001" />
 			</geometry>
-			<material name="Green" />
+			<material name="gray" />
 		</visual>
 		<collision>
@@ -98,4 +104,5 @@
 				<mesh filename="package://x80sv_description/meshes/collada/erratic_caster_support_link.dae"/>
 			</geometry>
+     			<material name="gray"/>
 		</visual>
 		<collision>
@@ -133,5 +140,5 @@
 					<mesh filename="package://x80sv_description/meshes/collada/erratic_caster_wheel_link.dae"/>
 				</geometry>
-				<material name="Black"/>
+				<material name="gray"/>
 			</visual>
 			<collision>
@@ -154,90 +161,82 @@
 		<origin xyz="0.0 -0.15525 -0.129" rpy="0 0 0" />
 	</wheel>
- <link name="kinect_link">
-  <collision>
-   <origin xyz="0 0 0" rpy="0 0 0"/>
-   <geometry><cylinder radius="0.07" length="0.01" /></geometry>
-  </collision>
+<!--kinect link-->
+<joint type="fixed" name="kinect_link_glue">
+   <origin xyz="-0.155 0 0.312" rpy="0 0 0"/>   <!--setup 0 0 ${-0.5*M_PI}-->${-0.0557*M_PI}
+   <child link="kinect_link"/>
+   <parent link="base_link" />
+</joint>
+<link name="kinect_link">
   <visual>
-   <origin xyz="0 0 0" rpy="0 0 0"/>
-   <geometry><cylinder radius="0.07" length="0.01" /></geometry>
+    <geometry>
+      <box size="0.072 0.278 0.073" />
+    </geometry>
+    <material name="Black" />
   </visual>
   <inertial>
-   <mass value="0.1" />
-   <inertia ixx="0.0001" ixy="0" ixz="0" iyy="0.0001" iyz="0" izz="0.0001" />
+      <mass value="0.001" />
+      <origin xyz="0 0 0" />
+      <inertia ixx="0.001" ixy="0.0" ixz="0.0"
+               iyy="0.001" iyz="0.0"
+               izz="0.001" />
   </inertial>
- </link>
-    <!-- Laser is positioned 13 cm +/- 1 cm forward of the robot wheel axis and 19 cm above ground level.
-        The X axis of the laser points to the left. X of the robot itself is forwards.
-        The gmapping node expects scan data centered around x axis of scan. Scans are recorded from 0
-        to 360 degrees from -pi to pi. The modeled axis of the scanner points right. This is also used
-        as frame. The actual x-axis of the scanner points right. This is where the scan starts.
-        With x-axis pointing left, the data is centered around the x-axis!
-        Works for both real and simulated robot.
-    -->
-  <joint type="fixed" name="kinect_link_glue">
-   <origin xyz="-0.155 0 0.312" rpy="0 0 0"/>   <!--setup 0 0 ${-0.5*M_PI}-->${-0.0557*M_PI}
-  <child link="kinect_link"/>
-  <parent link="base_link" />
+</link>
+<!--kinect depth link-->
+<joint name="kinect_depth_joint" type="fixed">
+  <origin xyz="0 0.028 0" rpy="0 0 0" />
+  <parent link="kinect_link" />
+  <child link="kinect_depth_frame" />
+</joint>
+<link name="kinect_depth_frame">
+  <inertial>
+      <mass value="0.01" />
+      <origin xyz="0 0 0" />
+      <inertia ixx="0.001" ixy="0.0" ixz="0.0"
+               iyy="0.001" iyz="0.0"
+               izz="0.001" />
+  </inertial>
+</link>
+<joint name="depth_optical_joint" type="fixed">
+  <origin xyz="0 0 0" rpy="${-M_PI/2} 0 ${-M_PI/2}" />
+  <parent link="kinect_depth_frame" />
+  <child link="kinect_depth_optical_frame" />
+</joint>
+<link name="kinect_depth_optical_frame">
+  <inertial>
+      <mass value="0.001" />
+      <origin xyz="0 0 0" />
+      <inertia ixx="0.0001" ixy="0.0" ixz="0.0"
+               iyy="0.0001" iyz="0.0"
+               izz="0.0001" />
+  </inertial>
+</link>
+<!--kinect rgb link-->
+  <joint name="kinect_rgb_joint" type="fixed">
+    <origin xyz="0 -0.028 0" rpy="0 0 0" />
+    <parent link="kinect_link" />
+    <child link="kinect_rgb_frame" />
   </joint>
-<!-- plugins -->
-<!-- hokuyo -->
-   <gazebo reference="kinect_link">
-    <sensor type="ray" name="kinect_link_sensor">
-      <pose>0 0 0 0 0 0</pose>
-	  <visualize>true</visualize>
-      <update_rate>10</update_rate>
-      <ray>
-        <scan>
-          <horizontal>
-            <samples>360</samples>
-            <resolution>1</resolution>
-            <!-- does not work: -->
-            <!--
-            <min_angle>0</min_angle>
-            <max_angle>${2*M_PI}</max_angle>
-            -->
-            <!-- works: -->
-            <min_angle>${-M_PI}</min_angle>
-            <max_angle>${M_PI}</max_angle>
-          </horizontal>
-        </scan>
-        <range>
-          <min>0.40</min>
-          <max>5.0</max>
-          <resolution>0.01</resolution>
-        </range>
-        <noise>
-          <type>gaussian</type>
-          <mean>0.0</mean>
-          <stddev>0.01</stddev>
-        </noise>
-      </ray>
-      <plugin name="gazebo_ros_head_hokuyo_controller" filename="libgazebo_ros_laser.so">
-        <topicName>/laser/scan</topicName>
-        <frameName>kinect_link</frameName>
-      </plugin>
-    </sensor>
-   </gazebo>
-<gazebo>
-	<plugin name="differential_drive_controller" filename="libgazebo_ros_diff_drive.so">
-		<alwaysOn>true</alwaysOn>
-		<updateRate>100</updateRate>
-		<leftJoint>base_link_right_wheel_joint</leftJoint>
-		<rightJoint>base_link_left_wheel_joint</rightJoint>
-		<wheelSeparation>${wheel_distance}</wheelSeparation>
-		<wheelDiameter>${wheel_diameter}</wheelDiameter>
-		<wheelTorque>1</wheelTorque>
-		<wheelAcceleration>1</wheelAcceleration>
-		<commandTopic>cmd_vel</commandTopic>
-		<odometryTopic>odom</odometryTopic>
-		<odometryFrame>odom</odometryFrame>
-		<robotBaseFrame>base_footprint</robotBaseFrame>
-		<publishWheelTF>false</publishWheelTF>
-		<publishTf>1</publishTf>
-		<rosDebugLevel>na</rosDebugLevel>
-		<odometrySource>odom</odometrySource>
-		<publishWheelJointState>true</publishWheelJointState>
-	</plugin>
-</gazebo>
+  <link name="kinect_rgb_frame">
+    <inertial>
+      <mass value="0.001" />
+      <origin xyz="0 0 0" />
+      <inertia ixx="0.0001" ixy="0.0" ixz="0.0"
+        iyy="0.0001" iyz="0.0"
+        izz="0.0001" />
+    </inertial>
+  </link>
+  <joint name="kinect_rgb_optical_joint" type="fixed">
+    <origin xyz="0 0 0" rpy="${-M_PI/2} 0 ${-M_PI/2}" />
+    <parent link="kinect_rgb_frame" />
+    <child link="kinect_rgb_optical_frame" />
+  </joint>
+  <link name="kinect_rgb_optical_frame">
+    <inertial>
+      <mass value="0.001" />
+      <origin xyz="0 0 0" />
+      <inertia ixx="0.0001" ixy="0.0" ixz="0.0"
+        iyy="0.0001" iyz="0.0"
+        izz="0.0001" />
+    </inertial>
+  </link>
 </robot>

Commit message: Add files via upload

File: x80sv_description/urdf/x80sv.xacro (robot description, xacro)
@@ -1,9 +1,12 @@
 <?xml version='1.0' ?>
 <robot name="x80sv" xmlns:xacro="http://www.ros.org/wiki/xacro">
-	 <material name="Black">
+	 <material name="black">
            <color rgba="0 0 0 1"/>
          </material>
 	 <material name="gray">
            <color rgba="0.8 0.8 0.8 1"/>
+         </material>
+	 <material name="red">
+           <color rgba="1 0 0 1"/>
          </material>
 	<xacro:include filename="$(find x80sv_description)/urdf/wheel.xacro" />
@@ -163,5 +166,5 @@
 <!--kinect link-->
 <joint type="fixed" name="kinect_link_glue">
-   <origin xyz="-0.155 0 0.312" rpy="0 0 0"/>   <!--setup 0 0 ${-0.5*M_PI}-->${-0.0557*M_PI}
+   <origin xyz="-0.155 0 0.352" rpy="0 0 0"/>   <!--setup 0 0 ${-0.5*M_PI}-->${-0.0557*M_PI}
    <child link="kinect_link"/>
    <parent link="base_link" />
@@ -170,7 +173,7 @@
   <visual>
     <geometry>
-      <box size="0.072 0.278 0.073" />
+      <box size="0.066 0.249 0.067" />
     </geometry>
-    <material name="Black" />
+    <material name="black" />
   </visual>
   <inertial>
@@ -240,3 +243,24 @@
     </inertial>
   </link>
+<!--Aluminum extrusion-->
+<joint type="fixed" name="box_glue1">
+   <origin xyz="-0.155 0 0.173" rpy="0 0 0"/>
+   <child link="box_link_1"/>
+   <parent link="base_link" />
+</joint>
+<link name="box_link_1">
+  <visual>
+    <geometry>
+      <box size="0.02 0.319 0.291" />
+    </geometry>
+    <material name="gray" />
+  </visual>
+  <inertial>
+      <mass value="0.001" />
+      <origin xyz="0 0 0" />
+      <inertia ixx="0.001" ixy="0.0" ixz="0.0"
+               iyy="0.001" iyz="0.0"
+               izz="0.001" />
+  </inertial>
+</link>
 </robot>

Commit message: Add files via upload

File: x80sv_description/urdf/x80sv.xacro (robot description, xacro)
@@ -1,4 +1,5 @@
 <?xml version='1.0' ?>
 <robot name="x80sv" xmlns:xacro="http://www.ros.org/wiki/xacro">
+    <property name="M_PI" value="3.14159" />
 	 <material name="black">
            <color rgba="0 0 0 1"/>
@@ -10,5 +11,5 @@
            <color rgba="1 0 0 1"/>
          </material>
-	<xacro:include filename="$(find x80sv_description)/urdf/wheel.xacro" />
+<xacro:include filename="$(find x80sv_description)/urdf/wheel.xacro" />
  <!--
   Wheel inertia:
@@ -164,83 +165,4 @@
 		<origin xyz="0.0 -0.15525 -0.129" rpy="0 0 0" />
 	</wheel>
-<!--kinect link-->
-<joint type="fixed" name="kinect_link_glue">
-   <origin xyz="-0.155 0 0.352" rpy="0 0 0"/>   <!--setup 0 0 ${-0.5*M_PI}-->${-0.0557*M_PI}
-   <child link="kinect_link"/>
-   <parent link="base_link" />
-</joint>
-<link name="kinect_link">
-  <visual>
-    <geometry>
-      <box size="0.066 0.249 0.067" />
-    </geometry>
-    <material name="black" />
-  </visual>
-  <inertial>
-      <mass value="0.001" />
-      <origin xyz="0 0 0" />
-      <inertia ixx="0.001" ixy="0.0" ixz="0.0"
-               iyy="0.001" iyz="0.0"
-               izz="0.001" />
-  </inertial>
-</link>
-<!--kinect depth link-->
-<joint name="kinect_depth_joint" type="fixed">
-  <origin xyz="0 0.028 0" rpy="0 0 0" />
-  <parent link="kinect_link" />
-  <child link="kinect_depth_frame" />
-</joint>
-<link name="kinect_depth_frame">
-  <inertial>
-      <mass value="0.01" />
-      <origin xyz="0 0 0" />
-      <inertia ixx="0.001" ixy="0.0" ixz="0.0"
-               iyy="0.001" iyz="0.0"
-               izz="0.001" />
-  </inertial>
-</link>
-<joint name="depth_optical_joint" type="fixed">
-  <origin xyz="0 0 0" rpy="${-M_PI/2} 0 ${-M_PI/2}" />
-  <parent link="kinect_depth_frame" />
-  <child link="kinect_depth_optical_frame" />
-</joint>
-<link name="kinect_depth_optical_frame">
-  <inertial>
-      <mass value="0.001" />
-      <origin xyz="0 0 0" />
-      <inertia ixx="0.0001" ixy="0.0" ixz="0.0"
-               iyy="0.0001" iyz="0.0"
-               izz="0.0001" />
-  </inertial>
-</link>
-<!--kinect rgb link-->
-  <joint name="kinect_rgb_joint" type="fixed">
-    <origin xyz="0 -0.028 0" rpy="0 0 0" />
-    <parent link="kinect_link" />
-    <child link="kinect_rgb_frame" />
-  </joint>
-  <link name="kinect_rgb_frame">
-    <inertial>
-      <mass value="0.001" />
-      <origin xyz="0 0 0" />
-      <inertia ixx="0.0001" ixy="0.0" ixz="0.0"
-        iyy="0.0001" iyz="0.0"
-        izz="0.0001" />
-    </inertial>
-  </link>
-  <joint name="kinect_rgb_optical_joint" type="fixed">
-    <origin xyz="0 0 0" rpy="${-M_PI/2} 0 ${-M_PI/2}" />
-    <parent link="kinect_rgb_frame" />
-    <child link="kinect_rgb_optical_frame" />
-  </joint>
-  <link name="kinect_rgb_optical_frame">
-    <inertial>
-      <mass value="0.001" />
-      <origin xyz="0 0 0" />
-      <inertia ixx="0.0001" ixy="0.0" ixz="0.0"
-        iyy="0.0001" iyz="0.0"
-        izz="0.0001" />
-    </inertial>
-  </link>
 <!--Aluminum extrusion-->
 <joint type="fixed" name="box_glue1">
@@ -264,3 +186,61 @@
   </inertial>
 </link>
+<!--kinect link-->
+<joint type="fixed" name="kinect_link_glue">
+   <origin xyz="-0.155 0 0.3195" rpy="0 0 0"/>
+   <child link="kinect_link"/>
+   <parent link="base_link" />
+</joint>
+ 	<link name="kinect_link">
+            <inertial>
+                <origin xyz="0.066 0.249 0.067" rpy="0 0 0" /><!--setup 0 0 ${-0.5*M_PI}-->
+                <mass value="0.82085" />
+                <inertia ixx="0.0039702" ixy="0" ixz="0" iyy="0.00059235" iyz="0" izz="0.0041195" />
+            </inertial>
+            <visual>
+                <origin xyz="0 0 0" rpy="0 0 0" />
+                <geometry>
+                    <mesh filename="package://x80sv_description/meshes/kinect2.STL" />
+                </geometry>
+                <material name="">
+                    <color rgba="0.1 0.1 0.1 1" />
+                </material>
+            </visual>
+            <collision>
+                <origin xyz="0 0 0" rpy="0 0 0" />
+                <geometry>
+                    <mesh filename="package://x80sv_description/meshes/kinect2.STL" />
+                </geometry>
+            </collision>
+        </link>
+        <!-- kinect2 rgb sensor physical attachment -->
+        <joint name="kinect2_rgb_joint" type="fixed">
+            <origin xyz="0.032 -0.095 0.042015" rpy="0 0 0" />
+            <parent link="kinect_link" />
+            <child link="kinect2_rgb_link" />
+        </joint>
+        <link name="kinect2_rgb_link" />
+        <!-- kinect2 rgb sensor frame -->
+        <joint name="kinect2_rgb_optical_frame_joint" type="fixed">
+            <origin xyz="0 0 0" rpy="${-M_PI / 2.0} 0 ${-M_PI / 2.0}" />
+            <parent link="kinect2_rgb_link" />
+            <child link="kinect2_rgb_optical_frame" />
+        </joint>
+        <link name="kinect2_rgb_optical_frame" />
+        <!-- gazebo extensions -->
+        <xacro:kinect2_rgb_gazebo link_name="kinect2_rgb_link" frame_name="kinect2_rgb_optical_frame" camera_name="kinect_V2" />
+        <!-- kinect2 ir sensor physical attachment -->
+        <joint name="kinect2_ir_joint" type="fixed">
+            <origin xyz="0 0.05157 0" rpy="0 0 0" />
+            <parent link="kinect2_rgb_link" />
+            <child link="kinect2_ir_link" />
+        </joint>
+        <link name="kinect2_ir_link" />
+        <!-- kinect2 ir sensor frame -->
+        <joint name="kinect2_ir_optical_frame_joint" type="fixed">
+            <origin xyz="0 0 0" rpy="${-M_PI / 2.0} 0 ${-M_PI / 2.0}" />
+            <parent link="kinect2_ir_link" />
+            <child link="kinect2_ir_optical_frame" />
+        </joint>
+        <link name="kinect2_ir_optical_frame" />
 </robot>
