Commit message: 2020/02/19 add commit

File: x80sv_description/urdf/x80sv_kinect.xacro (robot description, xacro)
@@ -163,4 +163,83 @@
 		<origin xyz="0.0 -0.15525 -0.129" rpy="0 0 0" />
 	</wheel>
+<!-- new add -->
+	<!-- Aluminum extrusion -->
+	<joint type="fixed" name="box_glue1">
+		<origin xyz="-0.155 0 0.173" rpy="0 0 0" />
+		<child link="box_link_1" />
+		<parent link="base_link" />
+	</joint>
+	<link name="box_link_1">
+		<visual>
+			<geometry>
+				<box size="0.02 0.319 0.291" />
+			</geometry>
+			<material name="gray" />
+		</visual>
+		<!--inertial>
+			<mass value="0.001" />
+			<origin xyz="0 0 0" />
+			<inertia ixx="0.001" ixy="0.0" ixz="0.0" iyy="0.001" iyz="0.0" izz="0.001" />
+		</inertial-->
+	</link>
+	<!-- kinect link -->
+	<joint type="fixed" name="kinect_link_glue">
+		<origin xyz="-0.155 0 0.3195" rpy="0 0 0" />
+		<child link="kinect_link" />
+		<parent link="base_link" />
+	</joint>
+	<link name="kinect_link">
+		<inertial>
+			<origin xyz="0.066 0.249 0.067" rpy="0 0 ${-0.5*M_PI}" /> <!-- setup 0 0 ${-0.5*M_PI} -->
+			<mass value="0.82085" />
+			<inertia ixx="0.0039702" ixy="0" ixz="0" iyy="0.00059235" iyz="0" izz="0.0041195" />
+		</inertial>
+		<visual>
+			<origin xyz="0 0 0" rpy="0 0 0" />
+			<geometry>
+				<mesh filename="package://x80sv_description/meshes/kinect2.STL" />
+			</geometry>
+			<material name="">
+				<color rgba="0.1 0.1 0.1 1" />
+			</material>
+		</visual>
+		<collision>
+			<origin xyz="0 0 0" rpy="0 0 0" />
+			<geometry>
+				<mesh filename="package://x80sv_description/meshes/kinect2.STL" />
+			</geometry>
+		</collision>
+	</link>
+	<!-- kinect2 rgb sensor physical attachment -->
+	<joint name="kinect2_rgb_joint" type="fixed">
+		<origin xyz="0.032 -0.095 0.042015" rpy="0 0 0" />
+		<parent link="kinect_link" />
+		<child link="kinect2_rgb_link" />
+	</joint>
+	<link name="kinect2_rgb_link" />
+	<!-- kinect2 rgb sensor frame -->
+	<joint name="kinect2_rgb_optical_frame_joint" type="fixed">
+		<origin xyz="0 0 0" rpy="${-M_PI / 2.0} 0 ${-M_PI / 2.0}" />
+		<parent link="kinect2_rgb_link" />
+		<child link="kinect2_rgb_optical_frame" />
+	</joint>
+	<link name="kinect2_rgb_optical_frame" />
+	<!-- gazebo extensions -->
+	<kinect2_rgb_gazebo link_name="kinect2_rgb_link" frame_name="kinect2_rgb_optical_frame" camera_name="kinect_V2" />
+	<!-- kinect2 ir sensor physical attachment -->
+	<joint name="kinect2_ir_joint" type="fixed">
+		<origin xyz="0 0.05157 0" rpy="0 0 0" />
+		<parent link="kinect2_rgb_link" />
+		<child link="kinect2_ir_link" />
+	</joint>
+	<link name="kinect2_ir_link" />
+	<!-- kinect2 ir sensor frame -->
+	<joint name="kinect2_ir_optical_frame_joint" type="fixed">
+		<origin xyz="0 0 0" rpy="${-M_PI / 2.0} 0 ${-M_PI / 2.0}" />
+		<parent link="kinect2_ir_link" />
+		<child link="kinect2_ir_optical_frame" />
+	</joint>
+	<link name="kinect2_ir_optical_frame" />
+<!-- new add -->
 <!-- gazebo plugins -->
 <gazebo>
@@ -185,3 +264,45 @@
 	</plugin>
 </gazebo>
+<gazebo reference="kinect_link">
+    <sensor type="depth" name="camera1">
+        <always_on>1</always_on>
+        <visualize>true</visualize>
+        <camera>
+            <horizontal_fov>1.047</horizontal_fov>
+            <image>
+                <width>640</width>
+                <height>480</height>
+                <format>R8G8B8</format>
+            </image>
+            <depth_camera>
+            </depth_camera>
+            <clip>
+                <near>0.1</near>
+                <far>100</far>
+            </clip>
+        </camera>
+             <plugin name="camera_controller" filename="libgazebo_ros_openni_kinect.so">
+             <alwaysOn>true</alwaysOn>
+                <updateRate>10.0</updateRate>
+                <cameraName>kinect_rgb</cameraName>
+                <frameName>kinect_link</frameName>
+            <imageTopicName>kinect_rgb</imageTopicName>
+            <!--depthImageTopicName>depth/image_raw</depthImageTopicName>
+            <pointCloudTopicName>depth/points</pointCloudTopicName>
+            <cameraInfoTopicName>rgb/camera_info</cameraInfoTopicName>
+            <depthImageCameraInfoTopicName>depth/camera_info</depthImageCameraInfoTopicName>
+            <pointCloudCutoff>0.4</pointCloudCutoff>
+                <hackBaseline>0.07</hackBaseline>
+                <distortionK1>0.0</distortionK1>
+                <distortionK2>0.0</distortionK2>
+                <distortionK3>0.0</distortionK3>
+                <distortionT1>0.0</distortionT1>
+                <distortionT2>0.0</distortionT2-->
+            <CxPrime>0.0</CxPrime>
+            <Cx>0.0</Cx>
+            <Cy>0.0</Cy>
+            <focalLength>0.0</focalLength>
+            </plugin>
+    </sensor>
+</gazebo>
 </robot>
